Commit message: added support for multi docker contained robot control

File: description/urdf/ur10_robot.urdf.xacro (robot description, xacro)
@@ -19,5 +19,5 @@
   <joint name="worldstation" type="fixed">
     <parent link="world" />
-    <child link = "station" />
+    <child link = "stationn" />
     <origin xyz="0.0 0.0 0.0" rpy="0.0 0.0 0.0" />
   </joint>
