Commit message: removed support for multi docker contained robot control

File: description/urdf/ur10_joint_limited_robot.urdf.xacro (robot description, xacro)
@@ -21,3 +21,11 @@
     <origin xyz="0.0 0.0 0" rpy="0.0 0.0 0.0" />
   </joint>
+  <!--
+  <link name="TARS/world" />
+  <joint name="base_world_world" type="fixed">
+    <parent link="TARS/world" />
+    <child link = "world" />
+    <origin xyz="0.0 0.0 0" rpy="0.0 0.0 0.0" />
+  </joint>
+  -->
 </robot>
