Commit message: Calibrated OFTOOL and Engine based on pointcloud. Created launchfile for IPS testing

File: description/urdf/ur10_unification.urdf.xacro (robot description, xacro)
@@ -60,5 +60,5 @@
     <xacro:property name="wrist_3_length" value="${d6}" />
     <link name="station">
-      <visual>
+      <!--visual>
         <geometry>
           <mesh filename="package://ros1_unification_2019/description/unstruct_ptcl_meshes/unification_wo_tstool.stl" scale="1 1 1"/>
@@ -72,5 +72,5 @@
           <mesh filename="package://ros1_unification_2019/description/unstruct_ptcl_meshes/unification_wo_tstool.stl" scale="1 1 1"/>
         </geometry>
-      </collision>
+      </collision-->
     </link>
     <joint name="station_robot" type="fixed">

Commit message: working stuff

File: description/urdf/ur10_unification.urdf.xacro (robot description, xacro)
@@ -291,5 +291,5 @@
       <collision>
         <geometry>
-          <box size="0.01 0.01 0.01"/>
+          <box size="0.0 0.0 0.0"/>
         </geometry>
         <origin rpy="0 0 0" xyz="-0.01 0 0"/>

Commit message: photoneo ladderframe

File: description/urdf/ur10_unification.urdf.xacro (robot description, xacro)
@@ -316,4 +316,19 @@
       <child link="${prefix}tool0"/>
     </joint>
+    <link name="photoneo">
+      <visual>
+        <geometry>
+          <mesh filename="package://ros1_unification_2019/description/cad_meshes/photoneo.stl" scale="0.001 0.001 0.001"/>
+        </geometry>
+        <material name="LightGrey">
+          <color rgba="0.7 0.7 0.7 1.0"/>
+        </material>
+      </visual>
+    </link>
+    <joint name="photoneobase" type="fixed">
+      <origin xyz="-0.4 -0.47 -0.32" rpy="0 0 1.5707"/>
+      <parent link="${prefix}base_link"/>
+      <child link="photoneo"/>
+    </joint>
     <!-- Connect tool0_controller to base using floating joint -->
     <!--link name="tool0_controller"/>

Commit message: hopefully multiple people in rviz

File: description/urdf/ur10_unification.urdf.xacro (robot description, xacro)
@@ -331,4 +331,11 @@
       <child link="photoneo"/>
     </joint>
+    <link name="kinect">
+    </link>
+    <joint name="kinectworld" type="fixed">
+      <origin xyz="-2 0 2" rpy="1.5707 0 1.5707"/>
+      <parent link="${prefix}world"/>
+      <child link="kinect"/>
+    </joint>
     <!-- Connect tool0_controller to base using floating joint -->
     <!--link name="tool0_controller"/>

Commit message: Skovde pre June demo mess

File: description/urdf/ur10_unification.urdf.xacro (robot description, xacro)
@@ -334,5 +334,5 @@
     </link>
     <joint name="kinectworld" type="fixed">
-      <origin xyz="-2 0 2" rpy="1.5707 0 1.5707"/>
+      <origin xyz="-2.15 -0.45 2.2" rpy="2 0 1.5707"/>
       <parent link="${prefix}world"/>
       <child link="kinect"/>
